Commit message: add link lengths as properties in xacro

File: robot_data/za_description/urdf/za_macro.xacro (robot description, xacro)
@@ -2,4 +2,12 @@
 <robot xmlns:xacro="http://www.ros.org/wiki/xacro">
   <xacro:macro name="za_macro" params="prefix">
+    <xacro:property name="l1z" value="0.45"/>
+    <xacro:property name="l2x" value="0.025"/>
+    <xacro:property name="l3y" value="-0.001"/>
+    <xacro:property name="l3z" value="0.454"/>
+    <xacro:property name="l4z" value="0.035"/>
+    <xacro:property name="l5x" value="0.4195"/>
+    <xacro:property name="l5y" value="0.001"/>
+    <xacro:property name="l6x" value="0.1175"/>
     <!-- link list -->
     <link name="${prefix}base_link">
@@ -91,5 +99,5 @@
       <parent link="${prefix}base_link"/>
       <child link="${prefix}link_1"/>
-      <origin rpy="0.0 0.0 0.0" xyz="0 0 0.45"/>
+      <origin rpy="0.0 0.0 0.0" xyz="0 0 ${l1z}"/>
       <axis xyz="0 0 1"/>
       <limit effort="0" lower="${radians(-170)}" upper="${radians(170)}" velocity="${radians(150)}"/>
@@ -98,5 +106,5 @@
       <parent link="${prefix}link_1"/>
       <child link="${prefix}link_2"/>
-      <origin rpy="0.0 0.0 0.0" xyz="0.025 0 0.0"/>
+      <origin rpy="0.0 0.0 0.0" xyz="${l2x} 0 0.0"/>
       <axis xyz="0 1 0"/>
       <limit effort="0" lower="${radians(-100)}" upper="${radians(130)}" velocity="${radians(112.5)}"/>
@@ -105,5 +113,5 @@
       <parent link="${prefix}link_2"/>
       <child link="${prefix}link_3"/>
-      <origin rpy="0.0 0.0 0.0" xyz="0.0 -0.001 0.454"/>
+      <origin rpy="0.0 0.0 0.0" xyz="0.0 ${l3y} ${l3z}"/>
       <axis xyz="0 1 0"/>
       <limit effort="0" lower="${radians(-120)}" upper="${radians(65)}" velocity="${radians(150)}"/>
@@ -112,5 +120,5 @@
       <parent link="${prefix}link_3"/>
       <child link="${prefix}link_4"/>
-      <origin rpy="0.0 0.0 0.0" xyz="0.0 0.0 0.035"/>
+      <origin rpy="0.0 0.0 0.0" xyz="0.0 0.0 ${l4z}"/>
       <axis xyz="1 0 0"/>
       <limit effort="0" lower="${radians(-180)}" upper="${radians(180)}" velocity="${radians(204.5)}"/>
@@ -119,5 +127,5 @@
       <parent link="${prefix}link_4"/>
       <child link="${prefix}link_5"/>
-      <origin rpy="0.0 0.0 0.0" xyz="0.4195 0.001 0.0"/>
+      <origin rpy="0.0 0.0 0.0" xyz="${l5x} ${l5y} 0.0"/>
       <axis xyz="0 1 0"/>
       <limit effort="0" lower="${radians(-140)}" upper="${radians(140)}" velocity="${radians(225)}"/>
@@ -126,5 +134,5 @@
       <parent link="${prefix}link_5"/>
       <child link="${prefix}link_6"/>
-      <origin rpy="0.0 0.0 0.0" xyz="0.1175 0.0 0.0"/>
+      <origin rpy="0.0 0.0 0.0" xyz="${l6x} 0.0 0.0"/>
       <axis xyz="1 0 0"/>
       <limit effort="0" lower="${radians(-360)}" upper="${radians(360)}" velocity="${radians(360)}"/>
